File: tutorial_LED_switch.kicad_pcb (KiCad board)
At the start: 2 copper layers, 50 x 50 mm, 4 parts, among them J1 Screw_Terminal_01x02, SW1 SW_SPST

Commit message: test commit
Other:
- board text added: "My First PCB test :)"
- board text removed: "My First PCB :)"
Changed lines of the file:
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@@
 		(layer "Edge.Cuts")
 	)
-	(gr_text "My First PCB :)"
+	(gr_text "My First PCB test :)"
 		(at 83.5 116 0)
 		(layer "F.SilkS")
